Commit message: 20260608

File: config/piper/piper_description.urdf (robot description, URDF)
Before this commit: robot piper, 11 links, 10 joints
Links:
- removed link dummy_link
- removed link gripper_base
- removed link link7
- removed link link8
- added link world
- link base_link: geometry collision mesh filename=package://agx_arm_description/agx_arm_urdf/piper/meshes/bas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; visual mesh filename=package://agx_arm_description/agx_arm_urdf/piper/meshes/dae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
- link link1: geometry collision mesh filename=package://agx_arm_description/agx_arm_urdf/piper/meshes/lin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; visual mesh filename=package://agx_arm_description/agx_arm_urdf/piper/meshes/dae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
- link link2: mass 1.17 -> 1.16; geometry collision mesh filename=package://agx_arm_description/agx_arm_urdf/piper/meshes/lin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; visual mesh filename=package://agx_arm_description/agx_arm_urdf/piper/meshes/dae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
- link link3: geometry collision mesh filename=package://agx_arm_description/agx_arm_urdf/piper/meshes/lin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; visual mesh filename=package://agx_arm_description/agx_arm_urdf/piper/meshes/dae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
- link link4: geometry collision mesh filename=package://agx_arm_description/agx_arm_urdf/piper/meshes/lin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; visual mesh filename=package://agx_arm_description/agx_arm_urdf/piper/meshes/dae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
- link link5: geometry collision mesh filename=package://agx_arm_description/agx_arm_urdf/piper/meshes/lin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; visual mesh filename=package://agx_arm_description/agx_arm_urdf/piper/meshes/dae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
- link link6: geometry collision mesh filename=package://agx_arm_description/agx_arm_urdf/piper/meshes/lin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; visual mesh filename=package://agx_arm_description/agx_arm_urdf/piper/meshes/dae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
Joints:
- removed joint base_to_dummy
- removed joint joint6_to_gripper_base
- removed joint joint7
- removed joint joint8
- added joint world_to_base_link: type fixed, parent world, child base_link, origin xyz=0 0 0 rpy=0 0 0
- joint joint1: limit lower=-2.618 upper=2.618 effort=100 velocity=5 -> lower=-2.6179938 upper=2.6179938 effort=100 velocity=5
- joint joint2: limit lower=0 upper=3.14 effort=100 velocity=5 -> lower=0 upper=3.1415926 effort=100 velocity=5; origin xyz=0 0 0 rpy=1.5708 -0.1359 -3.1416 -> xyz=0 0 0 rpy=1.5707963 -0.1357866 -3.1415926
- joint joint3: limit lower=-2.967 upper=0 effort=100 velocity=5 -> lower=-2.9670597 upper=0 effort=100 velocity=5; origin xyz=0.28503 0 0 rpy=0 0 -1.7939 -> xyz=0.28503 0 0 rpy=0 0 -1.7938494
- joint joint4: limit lower=-1.745 upper=1.745 effort=100 velocity=5 -> lower=-1.7453292 upper=1.7453292 effort=100 velocity=5; origin xyz=-0.021984 -0.25075 0 rpy=1.5708 0 0 -> xyz=-0.02198 -0.25075 0 rpy=1.5707963 0 0
- joint joint5: limit lower=-1.22 upper=1.22 effort=100 velocity=5 -> lower=-1.2217304 upper=1.2217304 effort=100 velocity=5; origin xyz=0 0 0 rpy=-1.5708 0 0 -> xyz=0 0 0 rpy=-1.5707963 0 0
- joint joint6: limit lower=-2.0944 upper=2.0944 effort=100 velocity=3 -> lower=-2.0943951 upper=2.0943951 effort=100 velocity=5; origin xyz=8.8259E-05 -0.091 0 rpy=1.5708 0 0 -> xyz=8.8259E-05 -0.091 0 rpy=1.5707963 0 0
